Commit message: add vision module 'no gripper' configuration

File: kinova_description/urdf/kinova_inertial.xacro (robot description, xacro)
@@ -28,4 +28,5 @@
    finger_proximal		57
    finger_distal      58
+   vision_module      59
 -->
 <xacro:macro name="inertia_cylinder" params="mass height radius axis:=0">
@@ -170,4 +171,13 @@
     </inertial>
   </xacro:unless>
+  <!-- vision_module = 59 -->
+  <!-- TODO edit this to match reality -->
+  <xacro:unless value="${mesh_no - 59}">
+    <inertial>
+        <mass value="0.01" />
+        <origin xyz="0.022 0 0" />
+        <xacro:inertia_cylinder height="0.03"  radius = "0.004" mass="0.01"/>
+    </inertial>
+  </xacro:unless>
 </xacro:macro>
 </root>

Commit message: add visual module urdf

File: kinova_description/urdf/kinova_inertial.xacro (robot description, xacro)
@@ -175,7 +175,7 @@
   <xacro:unless value="${mesh_no - 59}">
     <inertial>
-        <mass value="0.01" />
-        <origin xyz="0.022 0 0" />
-        <xacro:inertia_cylinder height="0.03"  radius = "0.004" mass="0.01"/>
+        <mass value="0.99" />
+        <origin xyz="0 0 -0.06" />
+        <xacro:inertia_cylinder height="0.03"  radius = "0.04" mass="0.727"/>
     </inertial>
   </xacro:unless>
